File: xfunctions.kicad_pcb (KiCad board)
At the start: 2 copper layers, 0 parts

Commit message: PCB 작성 완료
Parts:
- added D0: D_Small, Diode_SMD:D_SOD-323, B.Cu at (42.3, 52.4)
- added D1: D_Small, Diode_SMD:D_SOD-323, B.Cu at (61.3, 52.4)
- added D10: D_Small, Diode_SMD:D_SOD-323, B.Cu at (80.4, 71.4)
- added D11: D_Small, Diode_SMD:D_SOD-323, B.Cu at (99.4, 71.4)
- added D12: D_Small, Diode_SMD:D_SOD-323, B.Cu at (118.5, 71.4)
- added D13: D_Small, Diode_SMD:D_SOD-323, B.Cu at (137.5, 71.4)
- added D14: D_Small, Diode_SMD:D_SOD-323, B.Cu at (156.6, 71.4)
- added D15: D_Small, Diode_SMD:D_SOD-323, B.Cu at (175.6, 71.4)
- added D2: D_Small, Diode_SMD:D_SOD-323, B.Cu at (80.4, 52.4)
- added D3: D_Small, Diode_SMD:D_SOD-323, B.Cu at (99.4, 52.4)
- added D4: D_Small, Diode_SMD:D_SOD-323, B.Cu at (118.5, 52.4)
- added D5: D_Small, Diode_SMD:D_SOD-323, B.Cu at (137.5, 52.4)
- added D6: D_Small, Diode_SMD:D_SOD-323, B.Cu at (156.6, 52.4)
- added D7: D_Small, Diode_SMD:D_SOD-323, B.Cu at (175.6, 52.4)
- added D8: D_Small, Diode_SMD:D_SOD-323, B.Cu at (42.3, 71.4)
- added D9: D_Small, Diode_SMD:D_SOD-323, B.Cu at (61.3, 71.4)
- added SW0: SW_Push, PCM_marbastlib-mx:SW_MX_HS_CPG151101S11_1u, B.Cu at (47.6, 47.6)
- added SW1: SW_Push, PCM_marbastlib-mx:SW_MX_HS_CPG151101S11_1u, B.Cu at (66.7, 47.6)
- added SW10: SW_Push, PCM_marbastlib-mx:SW_MX_HS_CPG151101S11_1u, B.Cu at (85.7, 66.7)
- added SW11: SW_Push, PCM_marbastlib-mx:SW_MX_HS_CPG151101S11_1u, B.Cu at (104.8, 66.7)
- added SW12: SW_Push, PCM_marbastlib-mx:SW_MX_HS_CPG151101S11_1u, B.Cu at (123.8, 66.7)
- added SW13: SW_Push, PCM_marbastlib-mx:SW_MX_HS_CPG151101S11_1u, B.Cu at (142.9, 66.7)
- added SW14: SW_Push, PCM_marbastlib-mx:SW_MX_HS_CPG151101S11_1u, B.Cu at (161.9, 66.7)
- added SW15: SW_Push, PCM_marbastlib-mx:SW_MX_HS_CPG151101S11_1u, B.Cu at (181.0, 66.7)
- added SW2: SW_Push, PCM_marbastlib-mx:SW_MX_HS_CPG151101S11_1u, B.Cu at (85.7, 47.6)
- added SW3: SW_Push, PCM_marbastlib-mx:SW_MX_HS_CPG151101S11_1u, B.Cu at (104.8, 47.6)
- added SW4: SW_Push, PCM_marbastlib-mx:SW_MX_HS_CPG151101S11_1u, B.Cu at (123.8, 47.6)
- added SW5: SW_Push, PCM_marbastlib-mx:SW_MX_HS_CPG151101S11_1u, B.Cu at (142.9, 47.6)
- added SW6: SW_Push, PCM_marbastlib-mx:SW_MX_HS_CPG151101S11_1u, B.Cu at (161.9, 47.6)
- added SW7: SW_Push, PCM_marbastlib-mx:SW_MX_HS_CPG151101S11_1u, B.Cu at (181.0, 47.6)
- added SW8: SW_Push, PCM_marbastlib-mx:SW_MX_HS_CPG151101S11_1u, B.Cu at (47.6, 66.7)
- added SW9: SW_Push, PCM_marbastlib-mx:SW_MX_HS_CPG151101S11_1u, B.Cu at (66.7, 66.7)
- added U1: ProMicro, PCM_marbastlib-xp-promicroish:ProMicro_USBup, F.Cu at (201.9, 58.4)
- added U2: 74HC4051, Package_SO:SO-16_3.9x9.9mm_P1.27mm, B.Cu at (201.9, 57.1)
Routing:
- net COL_00: track 0.00 -> 208.4 mm, vias 0 -> 3
- net COL_01: track 0.00 -> 190.0 mm, vias 0 -> 3
- net COL_02: track 0.00 -> 172.8 mm, vias 0 -> 3
- net COL_03: track 0.00 -> 154.4 mm, vias 0 -> 3
- net ROW_00: track 0.00 -> 152.5 mm
- net ROW_01: track 0.00 -> 152.1 mm
- net COL_04: track 0.00 -> 133.3 mm, vias 0 -> 3
- net COL_05: track 0.00 -> 112.0 mm, vias 0 -> 3
- net COL_06: track 0.00 -> 90.7 mm, vias 0 -> 3
- net COL_07: track 0.00 -> 69.3 mm, vias 0 -> 3
- net VCC: track 0.00 -> 11.8 mm
- net Net-(D15-A): track 0.00 -> 7.08 mm
- net Net-(D14-A): track 0.00 -> 7.08 mm
- net Net-(D13-A): track 0.00 -> 7.08 mm
- net Net-(D7-A): track 0.00 -> 7.08 mm
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- added copper zone on F.Cu, net GND
Other:
- board outline added: 184.5 x 50 mm
